Commit message: Task: implement collision scene objects and speaker

File: src/unitree_ros/robots/z1_description/xacro/robot.xacro (robot description, xacro)
@@ -7,5 +7,5 @@
     <link name="world"/>
     <joint name="base_static_joint" type="fixed">
-        <origin rpy="0 0 0" xyz="0 0 0"/>
+        <origin rpy="0 0 0" xyz="0 0 0.5334"/>
         <parent link="world"/>
         <child link="link00"/>
